File: sample_kicad/sample/sample.kicad_sch (KiCad schematic)
At the start: 0 parts

Commit message: feature: update kicad sample
- use a sample from the template to have some real schematics
Parts:
- added C1: 100n, symbol Device:C_Small
- added J1: GPIO, Connector_PinSocket_2.54mm:PinSocket_2x20_P2.54mm_Vertical, symbol Connector_Generic:Conn_02x20_Odd_Even
- added JP1: ID_WP, symbol Jumper:SolderJumper_2_Open
- added R1, R2: 3.9k, symbol Device:R_Small
- added U1: CAT24C256, symbol Memory_EEPROM:CAT24C256
Connections:
- new net: JP1.1 (A), U1.7 (WP)
- new net +3V3: C1.1, J1.1 (Pin_1), J1.17 (Pin_17), JP1.2 (B), R1.1, R2.1, U1.8 (VCC)
- new net +5V: J1.2 (Pin_2), J1.4 (Pin_4)
- new net GND: C1.2, J1.14 (Pin_14), J1.20 (Pin_20), J1.25 (Pin_25), J1.30 (Pin_30), J1.34 (Pin_34), J1.39 (Pin_39), J1.6 (Pin_6), J1.9 (Pin_9), U1.4 (GND)
- new net GPIO10/SPI0.MOSI: J1.19 (Pin_19)
- new net GPIO11/SPI0.SCLK: J1.23 (Pin_23)
- new net GPIO12/PWM0: J1.32 (Pin_32)
- new net GPIO13/PWM1: J1.33 (Pin_33)
- new net GPIO14/TXD0: J1.8 (Pin_8)
- new net GPIO15/RXD0: J1.10 (Pin_10)
- new net GPIO16: J1.36 (Pin_36)
- new net GPIO17: J1.11 (Pin_11)
- new net GPIO18/PCM.CLK: J1.12 (Pin_12)
- new net GPIO19/PCM.FS: J1.35 (Pin_35)
- new net GPIO20/PCM.DIN: J1.38 (Pin_38)
- new net GPIO21/PCM.DOUT: J1.40 (Pin_40)
- new net GPIO22: J1.15 (Pin_15)
- new net GPIO23: J1.16 (Pin_16)
- new net GPIO24: J1.18 (Pin_18)
- new net GPIO25: J1.22 (Pin_22)
- new net GPIO26: J1.37 (Pin_37)
- new net GPIO27: J1.13 (Pin_13)
- new net GPIO2/SDA1: J1.3 (Pin_3)
- new net GPIO3/SCL1: J1.5 (Pin_5)
- new net GPIO4/GPCLK0: J1.7 (Pin_7)
- new net GPIO5: J1.29 (Pin_29)
- new net GPIO6: J1.31 (Pin_31)
- new net GPIO7/SPI0.CE1: J1.26 (Pin_26)
- new net GPIO8/SPI0.CE0: J1.24 (Pin_24)
- new net GPIO9/SPI0.MISO: J1.21 (Pin_21)
- new net ID_SCL: J1.28 (Pin_28), R2.2, U1.6 (SCL)
- new net ID_SDA: J1.27 (Pin_27), R1.2, U1.5 (SDA)
- no-connect marks 0 -> 3
Other:
- note added: "Additional pin functions: https://pinout.xyz/"
- note added: "ID_SD and ID_SC PINS: These pins are reserved for HAT ID EEPROM. At boot time this I2C interface will be interrogated to look for an EEPROM that identifes the attached board and allows automagic setup of the GPIOs (and optionally, Linux drivers). Bridging JP1 enables write protection. DO NOT USE these pins for anything other than attaching an I2C ID EEPROM. Leave unconnected if ID EEPROM not requ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"
